Commit message: add glueing support to kinova launcher

File: urdf/i3dr_titania_kinova.urdf.xacro (robot description, xacro)
@@ -18,5 +18,5 @@
         <parent link="world" />
         <child link = "root" />
-        <origin xyz="0 0 0" rpy="0 0 0" />
+        <origin xyz="0 0 0.01" rpy="0 0 0" />
     </joint>
     <joint name="kinova_titania_joint" type="fixed">

Commit message: add joint control nodes for kinova

File: urdf/i3dr_titania_kinova.urdf.xacro (robot description, xacro)
@@ -20,6 +20,28 @@
         <origin xyz="0 0 0.01" rpy="0 0 0" />
     </joint>
+    <link name="ground_plane_box">
+        <visual>
+            <origin xyz="0 0 0" rpy="0 0 0"/>
+            <geometry>
+                <box size="1.0 1.0 0.5"/>
+            </geometry>
+            <material name="Grey">
+                <color rgba="0.7 0.7 0.7 1.0"/>
+            </material>
+        </visual>
+        <collision>
+            <origin xyz="0 0 0" rpy="0 0 0"/>
+            <geometry>
+                <box size="1.0 1.0 0.5"/>
+            </geometry>
+        </collision>
+    </link>
+    <joint name="ground_plane_box" type="fixed">
+        <parent link="world" />
+        <child link="ground_plane_box" />
+        <origin xyz="0 0 -0.25" rpy="0 0 0" />
+    </joint>
     <joint name="kinova_titania_joint" type="fixed">
-        <origin xyz="0 0 0.08" rpy="-1.57 0 1.57" />
+        <origin xyz="0 0 0.09" rpy="-1.57 0 1.57" />
         <parent link="$(arg arm_name)_end_effector" />
         <child link="$(arg camera_name)_base_link" />
